File: Models/ResistorString/ResistorString.kicad_pcb (KiCad board)
At the start: 2 copper layers, 9 x 10 mm, 3 parts

Commit message: Upload modified KiCad project
Parts:
- added J1: Conn_01x04_Pin, Connector_PinHeader_2.54mm:PinHeader_1x04_P2.54mm_Vertical, F.Cu at (152.5, 98.0)
- R1: value CRCW0603357RFKEA -> 357
- R2: value CRCW0603357RFKEAC -> 806; footprint CRCW0603357RFKEAC:RESC1608X55N -> CRCW0603806RFKEA:RESC1508X50N
- R3: value CRCW0603357RFKEAHP -> 499; footprint CRCW0603357RFKEAHP:RESC1608X55N -> CRCW0603499RFKEA:RESC1508X50N
- moved R3 38.1 mm to (156.5, 105.6), turned to -90 degrees
- moved R2 37.5 mm to (156.5, 101.8), turned to -90 degrees
- moved R1 36.8 mm to (156.5, 98.0), turned to -90 degrees
Connections:
- R1 pad 1: unconnected-(R1-Pad1) -> Net-(J1-Pin_1)
- R1 pad 2: unconnected-(R1-Pad2) -> Net-(J1-Pin_2)
- R2 pad 1: unconnected-(R2-Pad1) -> Net-(J1-Pin_2)
- R2 pad 2: unconnected-(R2-Pad2) -> Net-(J1-Pin_3)
- R3 pad 1: unconnected-(R3-Pad1) -> Net-(J1-Pin_3)
- R3 pad 2: unconnected-(R3-Pad2) -> Net-(J1-Pin_4)
Routing:
- net Net-(J1-Pin_2): track 0.00 -> 6.56 mm
- net Net-(J1-Pin_3): track 0.00 -> 6.55 mm
- net Net-(J1-Pin_4): track 0.00 -> 4.32 mm
- net Net-(J1-Pin_1): track 0.00 -> 4.32 mm
Other:
- board size 9 x 10 mm -> 8 x 12.5 mm
- rule pad_to_mask_clearance: 0 -> 0.0508
- board text added: "0"
- board text added: "0 mm"
- board text added: "0.0152 mm"
- board text added: "0.02"
- board text added: "0.0356 mm"
- board text added: "0.1524 mm / 0.1524 mm"
- board text added: "0.2540 mm"
- board text added: "1"
- board text added: "1.524 mm"
- board text added: "1.6256 mm"
- board text added: "2"
- board text added: "3.3"
- board text added: "4.5"
- board text added: "8.0000 mm x 12.5000 mm"
- board text added: "B.Cu"
- board text added: "B.Mask"
- board text added: "B.Paste"
- board text added: "B.Silkscreen"
- board text added: "BOARD CHARACTERISTICS"
- board text added: "Board Thickness:"
- board text added: "Board overall dimensions:"
- board text added: "Bottom Silk Screen"
- board text added: "Bottom Solder Mask"
- board text added: "Bottom Solder Paste"
- board text added: "Castellated pads:"
- board text added: "Color"
- board text added: "Copper Finish:"
- board text added: "Copper Layer Count:"
- board text added: "Dielectric 1"
- board text added: "Edge card connectors:"
- board text added: "Epsilon R"
- board text added: "F.Cu"
- board text added: "F.Mask"
- board text added: "F.Paste"
- board text added: "F.Silkscreen"
- board text added: "FR4"
- board text added: "Impedance Control:"
- board text added: "Layer Name"
- board text added: "Loss Tangent"
- board text added: "Material"
- board text added: "Min hole diameter:"
- board text added: "Min track/spacing:"
- board text added: "No"
- board text added: "None"
- board text added: "Not specified"
- board text added: "Plated Board Edge:"
- board text added: "Thickness (mm)"
- board text added: "Top Silk Screen"
- board text added: "Top Solder Mask"
- board text added: "Top Solder Paste"
- board text added: "Type"
- board text added: "copper"
- board text added: "core"
